Commit message: Apply offset to joints to match initial condition

File: rrbot_description/urdf/rrbot.xacro (robot description, xacro)
@@ -1,5 +1,5 @@
 <?xml version="1.0"?>
 <!-- Revolute-Revolute Manipulator -->
-<robot name="rrbot" xmlns:xacro="http://www.ros.org/wiki/xacro">
+<robot name="rrbot" xmlns:xacro="http://ros.org/wiki/xacro">
   <!-- Constants for robot dimensions -->
   <xacro:property name="mass" value="1" /> <!-- arbitrary value for mass -->
@@ -12,5 +12,5 @@
   <xacro:include filename="$(find rrbot_description)/urdf/rrbot.gazebo" />
   <!-- Import Rviz colors -->
-  <xacro:include filename="$(find rrbot_description)/urdf/materials.xacro" />
+  <xacro:include filename="$(find rrbot_description)/urdf/extras.xacro" />
   <!-- Used for fixing robot to Gazebo 'base_link' -->
   <link name="world"/>
@@ -34,17 +34,12 @@
       <material name="orange"/>
     </visual>
-    <inertial>
+    <xacro:inertial_cuboid_with_pose mass="${mass}" x_length="${width}" y_length="${width}" z_length="${height1}">
       <origin xyz="0 0 ${height1/2}" rpy="0 0 0"/>
-      <mass value="${mass}"/>
-      <inertia
-        ixx="${mass / 12.0 * (width*width + height1*height1)}" ixy="0.0" ixz="0.0"
-        iyy="${mass / 12.0 * (height1*height1 + width*width)}" iyz="0.0"
-        izz="${mass / 12.0 * (width*width + width*width)}"/>
-    </inertial>
+    </xacro:inertial_cuboid_with_pose>
   </link>
   <joint name="joint1" type="continuous">
     <parent link="link1"/>
     <child link="link2"/>
-    <origin xyz="0 ${width} ${height1 - axel_offset}" rpy="0 0 0"/>
+    <origin xyz="0 ${width} ${height1 - axel_offset}" rpy="0 ${pi} 0"/>
     <axis xyz="0 1 0"/>
     <dynamics damping="0.7"/>
@@ -53,5 +48,5 @@
   <link name="link2">
     <collision>
-      <origin xyz="0 0 ${height2/2 - axel_offset}" rpy="0 0 0"/>
+      <origin xyz="0 0 ${height2/2 - axel_offset}" rpy="0 ${-pi} 0"/>
       <geometry>
 	      <box size="${width} ${width} ${height2}"/>
@@ -59,5 +54,5 @@
     </collision>
     <visual>
-      <origin xyz="0 0 ${height2/2 - axel_offset}" rpy="0 0 0"/>
+      <origin xyz="0 0 ${height2/2 - axel_offset}" rpy="0 ${-pi} 0"/>
       <geometry>
 	      <box size="${width} ${width} ${height2}"/>
@@ -65,12 +60,7 @@
       <material name="black"/>
     </visual>
-    <inertial>
-      <origin xyz="0 0 ${height2/2 - axel_offset}" rpy="0 0 0"/>
-      <mass value="${mass}"/>
-      <inertia
-        ixx="${mass / 12.0 * (width*width + height2*height2)}" ixy="0.0" ixz="0.0"
-        iyy="${mass / 12.0 * (height2*height2 + width*width)}" iyz="0.0"
-        izz="${mass / 12.0 * (width*width + width*width)}"/>
-    </inertial>
+    <xacro:inertial_cuboid_with_pose mass="${mass}" x_length="${width}" y_length="${width}" z_length="${height2}">
+      <origin xyz="0 0 ${height2/2 - axel_offset}" rpy="0 ${-pi} 0"/>
+    </xacro:inertial_cuboid_with_pose>
   </link>
   <joint name="joint2" type="continuous">
@@ -96,12 +86,7 @@
       <material name="orange"/>
     </visual>
-    <inertial>
+    <xacro:inertial_cuboid_with_pose mass="${mass}" x_length="${width}" y_length="${width}" z_length="${height3}">
       <origin xyz="0 0 ${height3/2 - axel_offset}" rpy="0 0 0"/>
-      <mass value="${mass}"/>
-      <inertia
-        ixx="${mass / 12.0 * (width*width + height3*height3)}" ixy="0.0" ixz="0.0"
-        iyy="${mass / 12.0 * (height3*height3 + width*width)}" iyz="0.0"
-        izz="${mass / 12.0 * (width*width + width*width)}"/>
-    </inertial>
+    </xacro:inertial_cuboid_with_pose>
   </link>
   <!--

Commit message: Fix joint initial positions

File: rrbot_description/urdf/rrbot.xacro (robot description, xacro)
@@ -48,5 +48,5 @@
   <link name="link2">
     <collision>
-      <origin xyz="0 0 ${height2/2 - axel_offset}" rpy="0 ${-pi} 0"/>
+      <origin xyz="0 0 ${height2/2 - axel_offset}" rpy="0 0 0"/>
       <geometry>
 	      <box size="${width} ${width} ${height2}"/>
@@ -54,5 +54,5 @@
     </collision>
     <visual>
-      <origin xyz="0 0 ${height2/2 - axel_offset}" rpy="0 ${-pi} 0"/>
+      <origin xyz="0 0 ${height2/2 - axel_offset}" rpy="0 0 0"/>
       <geometry>
 	      <box size="${width} ${width} ${height2}"/>
@@ -61,5 +61,5 @@
     </visual>
     <xacro:inertial_cuboid_with_pose mass="${mass}" x_length="${width}" y_length="${width}" z_length="${height2}">
-      <origin xyz="0 0 ${height2/2 - axel_offset}" rpy="0 ${-pi} 0"/>
+      <origin xyz="0 0 ${height2/2 - axel_offset}" rpy="0 0 0"/>
     </xacro:inertial_cuboid_with_pose>
   </link>
